Commit message: Scaled URDF to correct sizing of the robotic hand

File: src/hands_one/urdf/hands_one.urdf (robot description, URDF)
Before this commit: robot hands_one, 44 links, 43 joints
Links:
- link IndexMechanism_link: geometry collision mesh filename=package://hands_one/meshes/AbductionMechanism.stl scale=0.01 0.01 0.01; visual mesh filename=package://hands_one/meshes/AbductionMechanism.stl scale=0.01 0.01 0.01
- link IndexServo_link: geometry collision mesh filename=package://hands_one/meshes/servo.stl scale=0.01 0.01 0.01; visual mesh filename=package://hands_one/meshes/servo.stl scale=0.01 0.01 0.01
- link Index_DistalGearbox_link: geometry collision mesh filename=package://hands_one/meshes/Gearbox1.stl scale=0.01 0.01 0.01; visual mesh filename=package://hands_one/meshes/Gearbox1.stl scale=0.01 0.01 0.01
- link Index_Distal_link: geometry collision mesh filename=package://hands_one/meshes/IndexDistalUpdated.stl scale=0.01 0.01 0.01; visual mesh filename=package://hands_one/meshes/IndexDistalUpdated.stl scale=0.01 0.01 0.01
- link Index_MiddleGearbox_link: geometry collision mesh filename=package://hands_one/meshes/Gearbox1.stl scale=0.01 0.01 0.01; visual mesh filename=package://hands_one/meshes/Gearbox1.stl scale=0.01 0.01 0.01
- link Index_Middle_link: geometry collision mesh filename=package://hands_one/meshes/IndexMiddleUpdated.stl scale=0.01 0.01 0.01; visual mesh filename=package://hands_one/meshes/IndexMiddleUpdated.stl scale=0.01 0.01 0.01
- link Index_ProximalGearbox_link: geometry collision mesh filename=package://hands_one/meshes/Gearbox1.stl scale=0.01 0.01 0.01; visual mesh filename=package://hands_one/meshes/Gearbox1.stl scale=0.01 0.01 0.01
- link Index_Proximal_link: geometry collision mesh filename=package://hands_one/meshes/IndexProximalUpdated.stl scale=0.01 0.01 0.01; visual mesh filename=package://hands_one/meshes/IndexProximalUpdated.stl scale=0.01 0.01 0.01
- link LittleMechanism_link: geometry collision mesh filename=package://hands_one/meshes/AbductionMechanism.stl scale=0.01 0.01 0.01; visual mesh filename=package://hands_one/meshes/AbductionMechanism.stl scale=0.01 0.01 0.01
- link LittleServo_link: geometry collision mesh filename=package://hands_one/meshes/servo.stl scale=0.01 0.01 0.01; visual mesh filename=package://hands_one/meshes/servo.stl scale=0.01 0.01 0.01
- link Little_DistalGearbox_link: geometry collision mesh filename=package://hands_one/meshes/Gearbox1.stl scale=0.01 0.01 0.01; visual mesh filename=package://hands_one/meshes/Gearbox1.stl scale=0.01 0.01 0.01
- link Little_Distal_link: geometry collision mesh filename=package://hands_one/meshes/IndexDistalUpdated.stl scale=0.01 0.01 0.01; visual mesh filename=package://hands_one/meshes/IndexDistalUpdated.stl scale=0.01 0.01 0.01
- link Little_MiddleGearbox_link: geometry collision mesh filename=package://hands_one/meshes/Gearbox1.stl scale=0.01 0.01 0.01; visual mesh filename=package://hands_one/meshes/Gearbox1.stl scale=0.01 0.01 0.01
- link Little_Middle_link: geometry collision mesh filename=package://hands_one/meshes/IndexMiddleUpdated.stl scale=0.01 0.01 0.01; visual mesh filename=package://hands_one/meshes/IndexMiddleUpdated.stl scale=0.01 0.01 0.01
- link Little_ProximalGearbox_link: geometry collision mesh filename=package://hands_one/meshes/Gearbox1.stl scale=0.01 0.01 0.01; visual mesh filename=package://hands_one/meshes/Gearbox1.stl scale=0.01 0.01 0.01
- link Little_Proximal_link: geometry collision mesh filename=package://hands_one/meshes/LittleProximalUpdated.stl scale=0.01 0.01 0.01; visual mesh filename=package://hands_one/meshes/LittleProximalUpdated.stl scale=0.01 0.01 0.01
- link MiddleMechanism_link: geometry collision mesh filename=package://hands_one/meshes/AbductionMechanism.stl scale=0.01 0.01 0.01; visual mesh filename=package://hands_one/meshes/AbductionMechanism.stl scale=0.01 0.01 0.01
- link MiddleServo_link: geometry collision mesh filename=package://hands_one/meshes/servo.stl scale=0.01 0.01 0.01; visual mesh filename=package://hands_one/meshes/servo.stl scale=0.01 0.01 0.01
- link Middle_DistalGearbox_link: geometry collision mesh filename=package://hands_one/meshes/Gearbox1.stl scale=0.01 0.01 0.01; visual mesh filename=package://hands_one/meshes/Gearbox1.stl scale=0.01 0.01 0.01
- link Middle_Distal_link: geometry collision mesh filename=package://hands_one/meshes/IndexDistalUpdated.stl scale=0.01 0.01 0.01; visual mesh filename=package://hands_one/meshes/IndexDistalUpdated.stl scale=0.01 0.01 0.01
- link Middle_MiddleGearbox_link: geometry collision mesh filename=package://hands_one/meshes/Gearbox1.stl scale=0.01 0.01 0.01; visual mesh filename=package://hands_one/meshes/Gearbox1.stl scale=0.01 0.01 0.01
- link Middle_Middle_link: geometry collision mesh filename=package://hands_one/meshes/IndexMiddleUpdated.stl scale=0.01 0.01 0.01; visual mesh filename=package://hands_one/meshes/IndexMiddleUpdated.stl scale=0.01 0.01 0.01
- link Middle_ProximalGearbox_link: geometry collision mesh filename=package://hands_one/meshes/Gearbox1.stl scale=0.01 0.01 0.01; visual mesh filename=package://hands_one/meshes/Gearbox1.stl scale=0.01 0.01 0.01
- link Middle_Proximal_link: geometry collision mesh filename=package://hands_one/meshes/IndexProximalUpdated.stl scale=0.01 0.01 0.01; visual mesh filename=package://hands_one/meshes/IndexProximalUpdated.stl scale=0.01 0.01 0.01
- link PalmBackCover_link: geometry collision mesh filename=package://hands_one/meshes/PalmBackCoverUpdated.stl scale=0.01 0.01 0.01; visual mesh filename=package://hands_one/meshes/PalmBackCoverUpdated.stl scale=0.01 0.01 0.01
- link PalmFrontCover_link: geometry collision mesh filename=package://hands_one/meshes/PalmFrontCover.stl scale=0.01 0.01 0.01; visual mesh filename=package://hands_one/meshes/PalmFrontCover.stl scale=0.01 0.01 0.01
- link PalmMid_link: geometry collision mesh filename=package://hands_one/meshes/PalmMid.stl scale=0.01 0.01 0.01; visual mesh filename=package://hands_one/meshes/PalmMid.stl scale=0.01 0.01 0.01
- link RingMechanism_link: geometry collision mesh filename=package://hands_one/meshes/AbductionMechanism.stl scale=0.01 0.01 0.01; visual mesh filename=package://hands_one/meshes/AbductionMechanism.stl scale=0.01 0.01 0.01
- link RingServo_link: geometry collision mesh filename=package://hands_one/meshes/servo.stl scale=0.01 0.01 0.01; visual mesh filename=package://hands_one/meshes/servo.stl scale=0.01 0.01 0.01
- link Ring_DistalGearbox_link: geometry collision mesh filename=package://hands_one/meshes/Gearbox1.stl scale=0.01 0.01 0.01; visual mesh filename=package://hands_one/meshes/Gearbox1.stl scale=0.01 0.01 0.01
- link Ring_Distal_link: geometry collision mesh filename=package://hands_one/meshes/IndexDistalUpdated.stl scale=0.01 0.01 0.01; visual mesh filename=package://hands_one/meshes/IndexDistalUpdated.stl scale=0.01 0.01 0.01
- link Ring_MiddleGearbox_link: geometry collision mesh filename=package://hands_one/meshes/Gearbox1.stl scale=0.01 0.01 0.01; visual mesh filename=package://hands_one/meshes/Gearbox1.stl scale=0.01 0.01 0.01
- link Ring_Middle_link: geometry collision mesh filename=package://hands_one/meshes/IndexMiddleUpdated.stl scale=0.01 0.01 0.01; visual mesh filename=package://hands_one/meshes/IndexMiddleUpdated.stl scale=0.01 0.01 0.01
- link Ring_ProximalGearbox_link: geometry collision mesh filename=package://hands_one/meshes/Gearbox1.stl scale=0.01 0.01 0.01; visual mesh filename=package://hands_one/meshes/Gearbox1.stl scale=0.01 0.01 0.01
- link Ring_Proximal_link: geometry collision mesh filename=package://hands_one/meshes/IndexProximalUpdated.stl scale=0.01 0.01 0.01; visual mesh filename=package://hands_one/meshes/IndexProximalUpdated.stl scale=0.01 0.01 0.01
- link ThumbMechanism_link: geometry collision mesh filename=package://hands_one/meshes/AbductionMechanism.stl scale=0.01 0.01 0.01; visual mesh filename=package://hands_one/meshes/AbductionMechanism.stl scale=0.01 0.01 0.01
- link ThumbServo_link: geometry collision mesh filename=package://hands_one/meshes/servo.stl scale=0.01 0.01 0.01; visual mesh filename=package://hands_one/meshes/servo.stl scale=0.01 0.01 0.01
- link Thumb_DistalGearbox_link: geometry collision mesh filename=package://hands_one/meshes/Gearbox1.stl scale=0.01 0.01 0.01; visual mesh filename=package://hands_one/meshes/Gearbox1.stl scale=0.01 0.01 0.01
- link Thumb_Distal_link: geometry collision mesh filename=package://hands_one/meshes/IndexDistalUpdated.stl scale=0.01 0.01 0.01; visual mesh filename=package://hands_one/meshes/IndexDistalUpdated.stl scale=0.01 0.01 0.01
- link Thumb_MiddleGearbox_link: geometry collision mesh filename=package://hands_one/meshes/Gearbox1.stl scale=0.01 0.01 0.01; visual mesh filename=package://hands_one/meshes/Gearbox1.stl scale=0.01 0.01 0.01
- link Thumb_Middle_link: geometry collision mesh filename=package://hands_one/meshes/IndexMiddleUpdated.stl scale=0.01 0.01 0.01; visual mesh filename=package://hands_one/meshes/IndexMiddleUpdated.stl scale=0.01 0.01 0.01
- link Thumb_ProximalGearbox_link: geometry collision mesh filename=package://hands_one/meshes/Gearbox1.stl scale=0.01 0.01 0.01; visual mesh filename=package://hands_one/meshes/Gearbox1.stl scale=0.01 0.01 0.01
- link Thumb_Proximal_link: geometry collision mesh filename=package://hands_one/meshes/ThumbProximal.stl scale=0.01 0.01 0.01; visual mesh filename=package://hands_one/meshes/ThumbProximal.stl scale=0.01 0.01 0.01
Joints:
- joint IndexMechanism_joint: origin xyz=5.4 17.5 0 rpy=-1.5708 -1.5708 0 -> xyz=0.054 0.175 0 rpy=-1.5708 -1.5708 0
- joint IndexServo_joint: origin xyz=37.5 21.25 -2.0 rpy=1.5708 0 1.5708 -> xyz=0.375 0.2125 -0.020 rpy=1.5708 0 1.5708
- joint Index_DistalGearbox_joint: origin xyz=0 37.6 0 rpy=0 1.5708 0 -> xyz=0 0.376 0 rpy=0 1.5708 0
- joint Index_Distal_joint: origin xyz=0 2.95 0 rpy=0 -1.57 0 -> xyz=0 0.0295 0 rpy=0 -1.57 0
- joint Index_MiddleGearbox_joint: origin xyz=0 -26.6 0 rpy=3.14159 -1.5708 0 -> xyz=0 -0.266 0 rpy=3.14159 -1.5708 0
- joint Index_Middle_joint: origin xyz=0 3 0 rpy=0 1.57 0 -> xyz=0 0.03 0 rpy=0 1.57 0
- joint Index_ProximalGearbox_joint: origin xyz=0 23.75 -3 rpy=0 -1.57 -3.14159 -> xyz=0 0.2375 -0.03 rpy=0 -1.57 -3.14159
- joint Index_Proximal_joint: origin xyz=0 -29.6 0 rpy=0 1.5708 0 -> xyz=0 -0.296 0 rpy=0 1.5708 0
- joint LittleMechanism_joint: origin xyz=5.4 17.5 0 rpy=-1.5708 -1.5708 0 -> xyz=0.054 0.175 0 rpy=-1.5708 -1.5708 0
- joint LittleServo_joint: origin xyz=-37.5 8.75 -2.0 rpy=1.5708 0 1.5708 -> xyz=-0.375 0.0875 -0.020 rpy=1.5708 0 1.5708
- joint Little_DistalGearbox_joint: origin xyz=0 37.6 0 rpy=0 1.5708 0 -> xyz=0 0.376 0 rpy=0 1.5708 0
- joint Little_Distal_joint: origin xyz=0 2.95 0 rpy=0 -1.57 0 -> xyz=0 0.0295 0 rpy=0 -1.57 0
- joint Little_MiddleGearbox_joint: origin xyz=0 -24.6 0 rpy=3.14159 -1.5708 0 -> xyz=0 -0.246 0 rpy=3.14159 -1.5708 0
- joint Little_Middle_joint: origin xyz=0 3 0 rpy=0 1.57 0 -> xyz=0 0.03 0 rpy=0 1.57 0
- joint Little_ProximalGearbox_joint: origin xyz=0 23.75 -3 rpy=0 -1.57 -3.14159 -> xyz=0 0.2375 -0.03 rpy=0 -1.57 -3.14159
- joint Little_Proximal_joint: origin xyz=0 -27.6 0 rpy=0 1.5708 0 -> xyz=0 -0.276 0 rpy=0 1.5708 0
- joint MiddleMechanism_joint: origin xyz=5.4 17.5 0 rpy=-1.5708 -1.5708 0 -> xyz=0.054 0.175 0 rpy=-1.5708 -1.5708 0
- joint MiddleServo_joint: origin xyz=12.5 28.75 -2.0 rpy=1.5708 0 1.5708 -> xyz=0.125 0.2875 -0.020 rpy=1.5708 0 1.5708
- joint Middle_DistalGearbox_joint: origin xyz=0 37.6 0 rpy=0 1.5708 0 -> xyz=0 0.376 0 rpy=0 1.5708 0
- joint Middle_Distal_joint: origin xyz=0 2.95 0 rpy=0 -1.57 0 -> xyz=0 0.0295 0 rpy=0 -1.57 0
- joint Middle_MiddleGearbox_joint: origin xyz=0 -26.6 0 rpy=3.14159 -1.5708 0 -> xyz=0 -0.266 0 rpy=3.14159 -1.5708 0
- joint Middle_Middle_joint: origin xyz=0 3 0 rpy=0 1.57 0 -> xyz=0 0.03 0 rpy=0 1.57 0
- joint Middle_ProximalGearbox_joint: origin xyz=0 23.75 -3 rpy=0 -1.57 -3.14159 -> xyz=0 0.2375 -0.03 rpy=0 -1.57 -3.14159
- joint Middle_Proximal_joint: origin xyz=0 -29.6 0 rpy=0 1.5708 0 -> xyz=0 -0.296 0 rpy=0 1.5708 0
- joint PalmBack_joint: origin xyz=0 -5.0 -7.5 rpy=0 0 0 -> xyz=0 -0.050 -0.075 rpy=0 0 0
- joint PalmFront_joint: origin xyz=0 -5.0 17.5 rpy=0 0 0 -> xyz=0 -0.050 0.175 rpy=0 0 0
- joint RingMechanism_joint: origin xyz=5.4 17.5 0 rpy=-1.5708 -1.5708 0 -> xyz=0.054 0.175 0 rpy=-1.5708 -1.5708 0
- joint RingServo_joint: origin xyz=-12.5 21.25 -2.0 rpy=1.5708 0 1.5708 -> xyz=-0.125 0.2125 -0.020 rpy=1.5708 0 1.5708
- joint Ring_DistalGearbox_joint: origin xyz=0 37.6 0 rpy=0 1.5708 0 -> xyz=0 0.376 0 rpy=0 1.5708 0
- joint Ring_Distal_joint: origin xyz=0 2.95 0 rpy=0 -1.57 0 -> xyz=0 0.0295 0 rpy=0 -1.57 0
- joint Ring_MiddleGearbox_joint: origin xyz=0 -26.6 0 rpy=3.14159 -1.5708 0 -> xyz=0 -0.266 0 rpy=3.14159 -1.5708 0
- joint Ring_Middle_joint: origin xyz=0 3 0 rpy=0 1.57 0 -> xyz=0 0.03 0 rpy=0 1.57 0
- joint Ring_ProximalGearbox_joint: origin xyz=0 23.75 -3 rpy=0 -1.57 -3.14159 -> xyz=0 0.2375 -0.03 rpy=0 -1.57 -3.14159
- joint Ring_Proximal_joint: origin xyz=0 -29.6 0 rpy=0 1.5708 0 -> xyz=0 -0.296 0 rpy=0 1.5708 0
- joint ThumbMechanism_joint: origin xyz=5.4 17.5 0 rpy=-1.5708 -1.5708 0 -> xyz=0.054 0.175 0 rpy=-1.5708 -1.5708 0
- joint ThumbServo_joint: origin xyz=19.24 -39.31 -2.0 rpy=1.5708 0 0.7854 -> xyz=0.1924 -0.3931 -0.020 rpy=1.5708 0 0.7854
- joint Thumb_DistalGearbox_joint: origin xyz=0 37.6 0 rpy=0 1.5708 0 -> xyz=0 0.376 0 rpy=0 1.5708 0
- joint Thumb_Distal_joint: origin xyz=0 2.95 0 rpy=0 -1.57 0 -> xyz=0 0.0295 0 rpy=0 -1.57 0
- joint Thumb_MiddleGearbox_joint: origin xyz=0 -24.1 0 rpy=3.14159 0 0 -> xyz=0 -0.241 0 rpy=3.14159 0 0
- joint Thumb_Middle_joint: origin xyz=0 3 0 rpy=0 1.57 0 -> xyz=0 0.03 0 rpy=0 1.57 0
- joint Thumb_ProximalGearbox_joint: origin xyz=0 23.75 -3 rpy=0 -1.57 -3.14159 -> xyz=0 0.2375 -0.03 rpy=0 -1.57 -3.14159
- joint Thumb_Proximal_joint: origin xyz=0 -27.1 0 rpy=0 1.5708 0 -> xyz=0 -0.271 0 rpy=0 1.5708 0
