Commit message: Updated robotic hand model, controller, and meshes

File: src/hands_one/urdf/hands_one.urdf (robot description, URDF)
Before this commit: robot hands_one, 44 links, 43 joints
Links:
- link IndexMechanism_link: geometry collision mesh filename=package://hands_one/meshes/AbductionMechanism.stl scale=0.001 0.001 0.001; visual mesh filename=package://hands_one/meshes/AbductionMechanism.stl scale=0.001 0.001 0.001
- link IndexServo_link: geometry collision mesh filename=package://hands_one/meshes/servo.stl scale=0.001 0.001 0.001; visual mesh filename=package://hands_one/meshes/servo.stl scale=0.001 0.001 0.001
- link Index_DistalGearbox_link: geometry collision mesh filename=package://hands_one/meshes/Gearbox1.stl scale=0.001 0.001 0.001; visual mesh filename=package://hands_one/meshes/Gearbox1.stl scale=0.001 0.001 0.001
- link Index_Distal_link: geometry collision mesh filename=package://hands_one/meshes/IndexDistalUpdated.stl scale=0.001 0.001 0.001; visual mesh filename=package://hands_one/meshes/IndexDistalUpdated.stl scale=0.001 0.001 0.001
- link Index_MiddleGearbox_link: geometry collision mesh filename=package://hands_one/meshes/Gearbox1.stl scale=0.001 0.001 0.001; visual mesh filename=package://hands_one/meshes/Gearbox1.stl scale=0.001 0.001 0.001
- link Index_Middle_link: geometry collision mesh filename=package://hands_one/meshes/IndexMiddleUpdated.stl scale=0.001 0.001 0.001; visual mesh filename=package://hands_one/meshes/IndexMiddleUpdated.stl scale=0.001 0.001 0.001
- link Index_ProximalGearbox_link: geometry collision mesh filename=package://hands_one/meshes/Gearbox1.stl scale=0.001 0.001 0.001; visual mesh filename=package://hands_one/meshes/Gearbox1.stl scale=0.001 0.001 0.001
- link Index_Proximal_link: geometry collision mesh filename=package://hands_one/meshes/IndexProximalUpdated.stl scale=0.001 0.001 0.001; visual mesh filename=package://hands_one/meshes/IndexProximalUpdated.stl scale=0.001 0.001 0.001
- link LittleMechanism_link: geometry collision mesh filename=package://hands_one/meshes/AbductionMechanism.stl scale=0.001 0.001 0.001; visual mesh filename=package://hands_one/meshes/AbductionMechanism.stl scale=0.001 0.001 0.001
- link LittleServo_link: geometry collision mesh filename=package://hands_one/meshes/servo.stl scale=0.001 0.001 0.001; visual mesh filename=package://hands_one/meshes/servo.stl scale=0.001 0.001 0.001
- link Little_DistalGearbox_link: geometry collision mesh filename=package://hands_one/meshes/Gearbox1.stl scale=0.001 0.001 0.001; visual mesh filename=package://hands_one/meshes/Gearbox1.stl scale=0.001 0.001 0.001
- link Little_Distal_link: geometry collision mesh filename=package://hands_one/meshes/IndexDistalUpdated.stl scale=0.001 0.001 0.001; visual mesh filename=package://hands_one/meshes/IndexDistalUpdated.stl scale=0.001 0.001 0.001
- link Little_MiddleGearbox_link: geometry collision mesh filename=package://hands_one/meshes/Gearbox1.stl scale=0.001 0.001 0.001; visual mesh filename=package://hands_one/meshes/Gearbox1.stl scale=0.001 0.001 0.001
- link Little_Middle_link: geometry collision mesh filename=package://hands_one/meshes/IndexMiddleUpdated.stl scale=0.001 0.001 0.001; visual mesh filename=package://hands_one/meshes/IndexMiddleUpdated.stl scale=0.001 0.001 0.001
- link Little_ProximalGearbox_link: geometry collision mesh filename=package://hands_one/meshes/Gearbox1.stl scale=0.001 0.001 0.001; visual mesh filename=package://hands_one/meshes/Gearbox1.stl scale=0.001 0.001 0.001
- link Little_Proximal_link: geometry collision mesh filename=package://hands_one/meshes/LittleProximalUpdated.stl scale=0.001 0.001 0.001; visual mesh filename=package://hands_one/meshes/LittleProximalUpdated.stl scale=0.001 0.001 0.001
- link MiddleMechanism_link: geometry collision mesh filename=package://hands_one/meshes/AbductionMechanism.stl scale=0.001 0.001 0.001; visual mesh filename=package://hands_one/meshes/AbductionMechanism.stl scale=0.001 0.001 0.001
- link MiddleServo_link: geometry collision mesh filename=package://hands_one/meshes/servo.stl scale=0.001 0.001 0.001; visual mesh filename=package://hands_one/meshes/servo.stl scale=0.001 0.001 0.001
- link Middle_DistalGearbox_link: geometry collision mesh filename=package://hands_one/meshes/Gearbox1.stl scale=0.001 0.001 0.001; visual mesh filename=package://hands_one/meshes/Gearbox1.stl scale=0.001 0.001 0.001
- link Middle_Distal_link: geometry collision mesh filename=package://hands_one/meshes/IndexDistalUpdated.stl scale=0.001 0.001 0.001; visual mesh filename=package://hands_one/meshes/IndexDistalUpdated.stl scale=0.001 0.001 0.001
- link Middle_MiddleGearbox_link: geometry collision mesh filename=package://hands_one/meshes/Gearbox1.stl scale=0.001 0.001 0.001; visual mesh filename=package://hands_one/meshes/Gearbox1.stl scale=0.001 0.001 0.001
- link Middle_Middle_link: geometry collision mesh filename=package://hands_one/meshes/IndexMiddleUpdated.stl scale=0.001 0.001 0.001; visual mesh filename=package://hands_one/meshes/IndexMiddleUpdated.stl scale=0.001 0.001 0.001
- link Middle_ProximalGearbox_link: geometry collision mesh filename=package://hands_one/meshes/Gearbox1.stl scale=0.001 0.001 0.001; visual mesh filename=package://hands_one/meshes/Gearbox1.stl scale=0.001 0.001 0.001
- link Middle_Proximal_link: geometry collision mesh filename=package://hands_one/meshes/IndexProximalUpdated.stl scale=0.001 0.001 0.001; visual mesh filename=package://hands_one/meshes/IndexProximalUpdated.stl scale=0.001 0.001 0.001
- link PalmBackCover_link: geometry collision mesh filename=package://hands_one/meshes/PalmBackCoverUpdated.stl scale=0.001 0.001 0.001; visual mesh filename=package://hands_one/meshes/PalmBackCoverUpdated.stl scale=0.001 0.001 0.001
- link PalmFrontCover_link: geometry collision mesh filename=package://hands_one/meshes/PalmFrontCover.stl scale=0.001 0.001 0.001; visual mesh filename=package://hands_one/meshes/PalmFrontCover.stl scale=0.001 0.001 0.001
- link PalmMid_link: geometry collision mesh filename=package://hands_one/meshes/PalmMidUpdated.stl scale=0.001 0.001 0.001; visual mesh filename=package://hands_one/meshes/PalmMidUpdated.stl scale=0.001 0.001 0.001
- link RingMechanism_link: geometry collision mesh filename=package://hands_one/meshes/AbductionMechanism.stl scale=0.001 0.001 0.001; visual mesh filename=package://hands_one/meshes/AbductionMechanism.stl scale=0.001 0.001 0.001
- link RingServo_link: geometry collision mesh filename=package://hands_one/meshes/servo.stl scale=0.001 0.001 0.001; visual mesh filename=package://hands_one/meshes/servo.stl scale=0.001 0.001 0.001
- link Ring_DistalGearbox_link: geometry collision mesh filename=package://hands_one/meshes/Gearbox1.stl scale=0.001 0.001 0.001; visual mesh filename=package://hands_one/meshes/Gearbox1.stl scale=0.001 0.001 0.001
- link Ring_Distal_link: geometry collision mesh filename=package://hands_one/meshes/IndexDistalUpdated.stl scale=0.001 0.001 0.001; visual mesh filename=package://hands_one/meshes/IndexDistalUpdated.stl scale=0.001 0.001 0.001
- link Ring_MiddleGearbox_link: geometry collision mesh filename=package://hands_one/meshes/Gearbox1.stl scale=0.001 0.001 0.001; visual mesh filename=package://hands_one/meshes/Gearbox1.stl scale=0.001 0.001 0.001
- link Ring_Middle_link: geometry collision mesh filename=package://hands_one/meshes/IndexMiddleUpdated.stl scale=0.001 0.001 0.001; visual mesh filename=package://hands_one/meshes/IndexMiddleUpdated.stl scale=0.001 0.001 0.001
- link Ring_ProximalGearbox_link: geometry collision mesh filename=package://hands_one/meshes/Gearbox1.stl scale=0.001 0.001 0.001; visual mesh filename=package://hands_one/meshes/Gearbox1.stl scale=0.001 0.001 0.001
- link Ring_Proximal_link: geometry collision mesh filename=package://hands_one/meshes/IndexProximalUpdated.stl scale=0.001 0.001 0.001; visual mesh filename=package://hands_one/meshes/IndexProximalUpdated.stl scale=0.001 0.001 0.001
- link ThumbMechanism_link: geometry collision mesh filename=package://hands_one/meshes/AbductionMechanism.stl scale=0.001 0.001 0.001; visual mesh filename=package://hands_one/meshes/AbductionMechanism.stl scale=0.001 0.001 0.001
- link ThumbServo_link: geometry collision mesh filename=package://hands_one/meshes/servo.stl scale=0.001 0.001 0.001; visual mesh filename=package://hands_one/meshes/servo.stl scale=0.001 0.001 0.001
- link Thumb_DistalGearbox_link: geometry collision mesh filename=package://hands_one/meshes/Gearbox1.stl scale=0.001 0.001 0.001; visual mesh filename=package://hands_one/meshes/Gearbox1.stl scale=0.001 0.001 0.001
- link Thumb_Distal_link: geometry collision mesh filename=package://hands_one/meshes/IndexDistalUpdated.stl scale=0.001 0.001 0.001; visual mesh filename=package://hands_one/meshes/IndexDistalUpdated.stl scale=0.001 0.001 0.001
- link Thumb_MiddleGearbox_link: geometry collision mesh filename=package://hands_one/meshes/Gearbox1.stl scale=0.001 0.001 0.001; visual mesh filename=package://hands_one/meshes/Gearbox1.stl scale=0.001 0.001 0.001
- link Thumb_Middle_link: geometry collision mesh filename=package://hands_one/meshes/IndexMiddleUpdated.stl scale=0.001 0.001 0.001; visual mesh filename=package://hands_one/meshes/IndexMiddleUpdated.stl scale=0.001 0.001 0.001
- link Thumb_ProximalGearbox_link: geometry collision mesh filename=package://hands_one/meshes/Gearbox1.stl scale=0.001 0.001 0.001; visual mesh filename=package://hands_one/meshes/Gearbox1.stl scale=0.001 0.001 0.001
- link Thumb_Proximal_link: geometry collision mesh filename=package://hands_one/meshes/ThumbProximal.stl scale=0.001 0.001 0.001; visual mesh filename=package://hands_one/meshes/ThumbProximal.stl scale=0.001 0.001 0.001
Joints:
- joint IndexMechanism_joint: limit lower=-1.57 upper=1.57 effort=1 velocity=1 -> lower=-0.52 upper=0.1 effort=1 velocity=1; origin xyz=0.054 0.175 0 rpy=-1.5708 -1.5708 0 -> xyz=0.0054 0.0175 0 rpy=-1.5708 -1.5708 0
- joint IndexServo_joint: origin xyz=0.375 0.2125 -0.020 rpy=1.5708 0 1.5708 -> xyz=0.0375 0.02125 -0.0020 rpy=1.5708 0 1.5708
- joint Index_DistalGearbox_joint: origin xyz=0 0.376 0 rpy=0 1.5708 0 -> xyz=0 0.0376 0 rpy=0 1.5708 0
- joint Index_Distal_joint: origin xyz=0 0.0295 0 rpy=0 -1.57 0 -> xyz=0 0.00295 0 rpy=0 -1.57 0
- joint Index_MiddleGearbox_joint: origin xyz=0 -0.266 0 rpy=3.14159 -1.5708 0 -> xyz=0 -0.0266 0 rpy=3.14159 -1.5708 0
- joint Index_Middle_joint: origin xyz=0 0.03 0 rpy=0 1.57 0 -> xyz=0 0.003 0 rpy=0 1.57 0
- joint Index_ProximalGearbox_joint: limit lower=0 upper=1.57 effort=1 velocity=1 -> lower=-0.3 upper=1.57 effort=1 velocity=1; origin xyz=0 0.2375 -0.03 rpy=0 -1.57 -3.14159 -> xyz=0 0.02375 -0.003 rpy=0 -1.57 -3.14159
- joint Index_Proximal_joint: origin xyz=0 -0.296 0 rpy=0 1.5708 0 -> xyz=0 -0.0296 0 rpy=0 1.5708 0
- joint LittleMechanism_joint: limit lower=-1.57 upper=1.57 effort=1 velocity=1 -> lower=-0.1 upper=0.52 effort=1 velocity=1; origin xyz=0.054 0.175 0 rpy=-1.5708 -1.5708 0 -> xyz=0.0054 0.0175 0 rpy=-1.5708 -1.5708 0
- joint LittleServo_joint: origin xyz=-0.375 0.0875 -0.020 rpy=1.5708 0 1.5708 -> xyz=-0.0375 0.00875 -0.0020 rpy=1.5708 0 1.5708
- joint Little_DistalGearbox_joint: origin xyz=0 0.376 0 rpy=0 1.5708 0 -> xyz=0 0.0376 0 rpy=0 1.5708 0
- joint Little_Distal_joint: origin xyz=0 0.0295 0 rpy=0 -1.57 0 -> xyz=0 0.00295 0 rpy=0 -1.57 0
- joint Little_MiddleGearbox_joint: origin xyz=0 -0.246 0 rpy=3.14159 -1.5708 0 -> xyz=0 -0.0246 0 rpy=3.14159 -1.5708 0
- joint Little_Middle_joint: origin xyz=0 0.03 0 rpy=0 1.57 0 -> xyz=0 0.003 0 rpy=0 1.57 0
- joint Little_ProximalGearbox_joint: limit lower=0 upper=1.57 effort=1 velocity=1 -> lower=-0.3 upper=1.57 effort=1 velocity=1; origin xyz=0 0.2375 -0.03 rpy=0 -1.57 -3.14159 -> xyz=0 0.02375 -0.003 rpy=0 -1.57 -3.14159
- joint Little_Proximal_joint: origin xyz=0 -0.276 0 rpy=0 1.5708 0 -> xyz=0 -0.0276 0 rpy=0 1.5708 0
- joint MiddleMechanism_joint: limit lower=-1.57 upper=1.57 effort=1 velocity=1 -> lower=-0.2 upper=0.2 effort=1 velocity=1; origin xyz=0.054 0.175 0 rpy=-1.5708 -1.5708 0 -> xyz=0.0054 0.0175 0 rpy=-1.5708 -1.5708 0
- joint MiddleServo_joint: origin xyz=0.125 0.2875 -0.020 rpy=1.5708 0 1.5708 -> xyz=0.0125 0.02875 -0.0020 rpy=1.5708 0 1.5708
- joint Middle_DistalGearbox_joint: origin xyz=0 0.376 0 rpy=0 1.5708 0 -> xyz=0 0.0376 0 rpy=0 1.5708 0
- joint Middle_Distal_joint: origin xyz=0 0.0295 0 rpy=0 -1.57 0 -> xyz=0 0.00295 0 rpy=0 -1.57 0
- joint Middle_MiddleGearbox_joint: origin xyz=0 -0.266 0 rpy=3.14159 -1.5708 0 -> xyz=0 -0.0266 0 rpy=3.14159 -1.5708 0
- joint Middle_Middle_joint: origin xyz=0 0.03 0 rpy=0 1.57 0 -> xyz=0 0.003 0 rpy=0 1.57 0
- joint Middle_ProximalGearbox_joint: limit lower=0 upper=1.57 effort=1 velocity=1 -> lower=-0.3 upper=1.57 effort=1 velocity=1; origin xyz=0 0.2375 -0.03 rpy=0 -1.57 -3.14159 -> xyz=0 0.02375 -0.003 rpy=0 -1.57 -3.14159
- joint Middle_Proximal_joint: origin xyz=0 -0.296 0 rpy=0 1.5708 0 -> xyz=0 -0.0296 0 rpy=0 1.5708 0
- joint PalmBack_joint: origin xyz=0 -0.050 -0.075 rpy=0 0 0 -> xyz=0 -0.0050 -0.0075 rpy=0 0 0
- joint PalmFront_joint: origin xyz=0 -0.050 0.175 rpy=0 0 0 -> xyz=0 -0.0050 0.0175 rpy=0 0 0
- joint RingMechanism_joint: limit lower=-1.57 upper=1.57 effort=1 velocity=1 -> lower=-0.1 upper=0.35 effort=1 velocity=1; origin xyz=0.054 0.175 0 rpy=-1.5708 -1.5708 0 -> xyz=0.0054 0.0175 0 rpy=-1.5708 -1.5708 0
- joint RingServo_joint: origin xyz=-0.125 0.2125 -0.020 rpy=1.5708 0 1.5708 -> xyz=-0.0125 0.02125 -0.0020 rpy=1.5708 0 1.5708
- joint Ring_DistalGearbox_joint: origin xyz=0 0.376 0 rpy=0 1.5708 0 -> xyz=0 0.0376 0 rpy=0 1.5708 0
- joint Ring_Distal_joint: origin xyz=0 0.0295 0 rpy=0 -1.57 0 -> xyz=0 0.00295 0 rpy=0 -1.57 0
- joint Ring_MiddleGearbox_joint: origin xyz=0 -0.266 0 rpy=3.14159 -1.5708 0 -> xyz=0 -0.0266 0 rpy=3.14159 -1.5708 0
- joint Ring_Middle_joint: origin xyz=0 0.03 0 rpy=0 1.57 0 -> xyz=0 0.003 0 rpy=0 1.57 0
- joint Ring_ProximalGearbox_joint: limit lower=0 upper=1.57 effort=1 velocity=1 -> lower=-0.3 upper=1.57 effort=1 velocity=1; origin xyz=0 0.2375 -0.03 rpy=0 -1.57 -3.14159 -> xyz=0 0.02375 -0.003 rpy=0 -1.57 -3.14159
- joint Ring_Proximal_joint: origin xyz=0 -0.296 0 rpy=0 1.5708 0 -> xyz=0 -0.0296 0 rpy=0 1.5708 0
- joint ThumbMechanism_joint: limit lower=-1.57 upper=1.57 effort=1 velocity=1 -> lower=-0.6 upper=1.1 effort=1 velocity=1; origin xyz=0.054 0.175 0 rpy=-1.5708 -1.5708 0 -> xyz=0.0054 0.0175 0 rpy=-1.5708 -1.5708 0
- joint ThumbServo_joint: origin xyz=0.1924 -0.3931 -0.020 rpy=1.5708 0 0.7854 -> xyz=0.01924 -0.03931 0.01795 rpy=1.5708 0 0.7854
- joint Thumb_DistalGearbox_joint: origin xyz=0 0.376 0 rpy=0 1.5708 0 -> xyz=0 0.0376 0 rpy=0 1.5708 0
- joint Thumb_Distal_joint: origin xyz=0 0.0295 0 rpy=0 -1.57 0 -> xyz=0 0.00295 0 rpy=0 -1.57 0
- joint Thumb_MiddleGearbox_joint: origin xyz=0 -0.241 0 rpy=3.14159 0 0 -> xyz=0 -0.0241 0 rpy=3.14159 0 0
- joint Thumb_Middle_joint: origin xyz=0 0.03 0 rpy=0 1.57 0 -> xyz=0 0.003 0 rpy=0 1.57 0
- joint Thumb_ProximalGearbox_joint: limit lower=0 upper=1.57 effort=1 velocity=1 -> lower=-1.0 upper=1.57 effort=1 velocity=1; origin xyz=0 0.2375 -0.03 rpy=0 -1.57 -3.14159 -> xyz=0 0.02375 -0.003 rpy=0 -1.57 -3.14159
- joint Thumb_Proximal_joint: origin xyz=0 -0.271 0 rpy=0 1.5708 0 -> xyz=0 -0.0271 0 rpy=0 1.5708 0

Commit message: final changes to improve code performance

File: src/hands_one/urdf/hands_one.urdf (robot description, URDF)
Before this commit: robot hands_one, 44 links, 43 joints
Links:
- added link world
Joints:
- added joint world_fixed: type fixed, parent world, child base_link, origin xyz=0 0 0.5 rpy=1.5708 0 0
